File: Ripwing.kicad_sch (KiCad schematic)
At the start: 65 parts, among them Q1 BSS138, SW1 SW_Push, U1 STM32H723VGTx, U2 LSM6DS0, U3 BMP581, U4 TLV75733PDBV, U5 USBLC6-2SC6, U6 MMC5983MA, Y2 ASE-xxxMHz

Commit message: schematic done (rage baited nerd)
Other:
- note added: "Bulk"
- moved on the sheet: 5Volt, BuzzerPad, C1, C10, C14, C15, C16, C17, C18, C19, C2, C20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
